File: tycho/vbus_switch.kicad_sch (KiCad schematic)
At the start: 11 parts, among them Q13 NPN, Q14 PMOS, Q3 PMOS, Q4 2PNP

Commit message: Update schematic and board with footprint changes.
Parts:
- Q14, Q3: footprint (none) -> tycho:PowerPAK-SC-70-6L
Connections:
- net VBUS_EUT: now also Q3.0 (D)
- net at D1.1 (K), Q14.1 (D), Q14.2 (D)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: now also Q14.0 (D)
Changed lines of the file:
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@@
       (effects (font (size 1.27 1.27)))
     )
-    (property "Footprint" "" (at 152.4 71.12 0)
+    (property "Footprint" "tycho:PowerPAK-SC-70-6L" (at 152.4 71.12 0)
       (effects (font (size 1.27 1.27)) hide)
     )
@@
     )
     (pin "7")
+    (pin "0")
     (pin "1")
     (pin "2")
@@
       (effects (font (size 1.27 1.27)))
     )
-    (property "Footprint" "" (at 113.03 71.12 0)
+    (property "Footprint" "tycho:PowerPAK-SC-70-6L" (at 113.03 71.12 0)
       (effects (font (size 1.27 1.27)) hide)
     )
@@
     )
     (pin "7")
+    (pin "0")
     (pin "1")
     (pin "2")

Commit message: Cleanup and DRC pass.
Parts:
- Q14, Q3: footprint tycho:PowerPAK-SC-70-6L -> Package_TO_SOT_SMD:Vishay_PowerPAK_SC70-6L_Single; symbol tycho:SiA469 -> Transistor_FET:SiA449DJ
Connections:
- net VBUS: no longer Q14.7 (S)
- net VBUS_EUT: no longer Q3.0 (D), Q3.2 (D), Q3.5 (D), Q3.6 (D)
- net at D1.1 (K), Q14.1 (D), Q3.4 (S)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: no longer Q14.0 (D), Q14.2 (D), Q14.5 (D), Q14.6 (D), Q3.7 (S)
Changed lines of the file:
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@@
     (effects (font (size 1.27 1.27)) (justify right))
   )
-  (symbol (lib_id "tycho:SiA469") (at 152.4 71.12 90) (unit 1)
+  (symbol (lib_id "Transistor_FET:SiA449DJ") (at 152.4 73.66 90) (unit 1)
     (in_bom yes) (on_board yes) (dnp no) (fields_autoplaced)
-    (property "Reference" "Q14" (at 152.4 62.9752 90)
+    (property "Reference" "Q14" (at 152.4 65.5152 90)
       (effects (font (size 1.27 1.27)))
     )
-    (property "Value" "PMOS" (at 152.4 65.5121 90)
+    (property "Value" "PMOS" (at 152.4 68.0521 90)
       (effects (font (size 1.27 1.27)))
     )
-    (property "Footprint" "tycho:PowerPAK-SC-70-6L" (at 152.4 71.12 0)
+    (property "Footprint" "Package_TO_SOT_SMD:Vishay_PowerPAK_SC70-6L_Single" (at 154.305 68.58 0)
+      (effects (font (size 1.27 1.27) italic) (justify left) hide)
+    )
+    (property "Datasheet" "https://www.vishay.com/docs/75354/sia469dj.pdf" (at 152.4 73.66 0)
       (effects (font (size 1.27 1.27)) hide)
     )
-    (property "Datasheet" "https://www.vishay.com/docs/75354/sia469dj.pdf" (at 152.4 71.12 0)
+    (property "Manufacturer" "Vishay Siliconix" (at 152.4 73.66 0)
       (effects (font (size 1.27 1.27)) hide)
     )
-    (property "Manufacturer" "Vishay Siliconix" (at 152.4 71.12 0)
+    (property "Part Number" "SIA469DJ-T1-GE3" (at 152.4 73.66 0)
       (effects (font (size 1.27 1.27)) hide)
     )
-    (property "Part Number" "SIA469DJ-T1-GE3" (at 152.4 71.12 0)
+    (property "Description" "MOSFET P-CH 30V 12A PPAK SC70-6" (at 152.4 73.66 0)
       (effects (font (size 1.27 1.27)) hide)
     )
-    (property "Description" "MOSFET P-CH 30V 12A PPAK SC70-6" (at 152.4 71.12 0)
-      (effects (font (size 1.27 1.27)) hide)
-    )
-    (pin "7")
-    (pin "0")
     (pin "1")
-    (pin "2")
     (pin "3")
     (pin "4")
-    (pin "5")
-    (pin "6")
     (instances
       (project "tycho"
@@
     )
   )
-  (symbol (lib_id "tycho:SiA469") (at 113.03 71.12 90) (unit 1)
+  (symbol (lib_id "Transistor_FET:SiA449DJ") (at 113.03 73.66 90) (unit 1)
     (in_bom yes) (on_board yes) (dnp no) (fields_autoplaced)
-    (property "Reference" "Q3" (at 113.03 62.9752 90)
+    (property "Reference" "Q3" (at 113.03 65.5152 90)
       (effects (font (size 1.27 1.27)))
     )
-    (property "Value" "PMOS" (at 113.03 65.5121 90)
+    (property "Value" "PMOS" (at 113.03 68.0521 90)
       (effects (font (size 1.27 1.27)))
     )
-    (property "Footprint" "tycho:PowerPAK-SC-70-6L" (at 113.03 71.12 0)
+    (property "Footprint" "Package_TO_SOT_SMD:Vishay_PowerPAK_SC70-6L_Single" (at 114.935 68.58 0)
+      (effects (font (size 1.27 1.27) italic) (justify left) hide)
+    )
+    (property "Datasheet" "https://www.vishay.com/docs/75354/sia469dj.pdf" (at 113.03 73.66 0)
       (effects (font (size 1.27 1.27)) hide)
     )
-    (property "Datasheet" "https://www.vishay.com/docs/75354/sia469dj.pdf" (at 113.03 71.12 0)
+    (property "Manufacturer" "Vishay Siliconix" (at 113.03 73.66 0)
       (effects (font (size 1.27 1.27)) hide)
     )
-    (property "Manufacturer" "Vishay Siliconix" (at 113.03 71.12 0)
+    (property "Part Number" "SIA469DJ-T1-GE3" (at 113.03 73.66 0)
       (effects (font (size 1.27 1.27)) hide)
     )
-    (property "Part Number" "SIA469DJ-T1-GE3" (at 113.03 71.12 0)
+    (property "Description" "MOSFET P-CH 30V 12A PPAK SC70-6" (at 113.03 73.66 0)
       (effects (font (size 1.27 1.27)) hide)
     )
-    (property "Description" "MOSFET P-CH 30V 12A PPAK SC70-6" (at 113.03 71.12 0)
-      (effects (font (size 1.27 1.27)) hide)
-    )
-    (pin "7")
-    (pin "0")
     (pin "1")
-    (pin "2")
     (pin "3")
     (pin "4")
-    (pin "5")
-    (pin "6")
     (instances
       (project "tycho"
